File: PCB/master/master.sch (EAGLE design)
At the start: 0 parts

Commit message: finished PCB designs
Parts:
- added A2: RPI3-B, RPI_HEADER_snapEDA:RPI3-B
- added C1, C3, C32, C33, C34, C35, C4, C5: 100nF 50V, rcl:C-EUC0805
- added C10, C2: 1uF 16V, rcl:C-EUC0805
- added C11, C12: 47u 10V, rcl:C-EUC1210
- added C13, C14: 100n 50V, rcl:C-EUC1206
- added C15, C16: 2u2 50V, rcl:C-EUC1206
- added C17, C18: (no value), rcl:CPOL-EUUD-5X5,8
- added C9: NM, rcl:C-EUC0805
- added D1, D3, D4, D5: CDSOT23-0502B, CDSOT23-SM712_snapEDA:CDSOT23-SM712
- added D2: B360B-13-F, diode:MBRS130LT3
- added D6: B260-13-F, diode:MBRS130LT3
- added F4: 40012000000, 400XXX0000:40012000000
- added L1: 10uH 3A9, parts:1217AS-H-100M=P3
- added LOGO1: OSHW_LOGO_FILLX0350-NT, ohw-logo:OSHW_LOGO_FILLX0350-NT
- added R1: B72214S0300K101, varistor:S14K300
- added R12, R13: 4k7, rcl:R-EU_R1206
- added R18, R20, R21, R23, R24, R26, R27, R29: 1k, rcl:R-EU_R1206
- added R19, R22, R25, R28: 120R, rcl:R-EU_R1206
- added R4: 41k2, rcl:R-EU_R1206
- added R5: 68k, rcl:R-EU_R1206
- added R6: 12k, rcl:R-EU_R1206
- added T1, T2, T3, T4: WJ500V-5.08-3P, parts:WJ500V-5.08-3P
- added U2: LMR16020, LMR160X0_snapEDA:LMR16020
- added U4, U5, U6, U7: SN65HVD11DR, SN65HVD11DR_snapEDA:SN65HVD11DR
- added U8: MAX14830ETMT, MAX14830ETMT_snapEDA:MAX14830ETMT
- added Y1: X1G004171001800 12MHz, X1G0041710033_snapEDA:X1G0041710033
Connections:
- new net +24V: C14.1, C15.1, C16.1, C17.+, C18.+, D6.C, U2.EN, U2.VIN
- new net +3V3: A2.3V3[1], A2.3V3[2], C3.1, C32.1, C33.1, C34.1, C35.1, C4.1, C5.1, R12.1, R13.1, R18.1, R21.1, R24.1, R27.1, U4.VCC, U5.VCC, U6.VCC, U7.VCC, U8.LDOEN, U8.SPI/*I2C, U8.VA, U8.VEXT, U8.VL, Y1.VCC
- new net +5V: A2.5V[1], A2.5V[2], C10.1, C11.1, C12.1, C9.1, L1.1, R5.1
- new net A0: D1.IO2, R18.2, R19.1, T1.1, U7.A
- new net A1: D3.IO2, R21.2, R22.1, T1.3, U6.A
- new net A2: D4.IO2, R24.2, R25.1, T3.1, U5.A
- new net A3: D5.IO2, R27.2, R28.1, T3.3, U4.A
- new net AS312_OUT: U8.*CTS0
- new net B0: D1.IO1, R19.2, R20.1, T1.2, U7.B
- new net B1: D3.IO1, R22.2, R23.1, T2.1, U6.B
- new net B2: D4.IO1, R25.2, R26.1, T3.2, U5.B
- new net B3: D5.IO1, R28.2, R29.1, T4.1, U4.B
- new net CLK_12M: U8.XIN, Y1.OUT
- new net GND: A2.GND[1], A2.GND[2], A2.GND[3], A2.GND[4], A2.GND[5], A2.GND[7], A2.GND[8], C1.2, C10.2, C11.2, C12.2, C14.2, C15.2, C16.2, C17.-, C18.-, C2.2, C3.2, C32.2, C33.2, C34.2, C35.2, C4.2, C5.2, D1.GND, D2.A, D3.GND, D4.GND, D5.GND, R1.1, R20.2, R23.2, R26.2, R29.2, R4.2, R6.2, T2.2, T4.2, U2.GND, U4.GND, U5.GND, U6.GND, U7.GND, U8.AGND, U8.DGND, U8.EP, Y1.GND
- new net MAX_IO0: U8.GPIO0
- new net MAX_IO1: U8.GPIO1
- new net MAX_IO10: U8.GPIO10
- new net MAX_IO11: U8.GPIO11
- new net MAX_IO12: U8.GPIO12
- new net MAX_IO13: U8.GPIO13
- new net MAX_IO14: U8.GPIO14
- new net MAX_IO15: U8.GPIO15
- new net MAX_IO2: U8.GPIO2
- new net MAX_IO3: U8.GPIO3
- new net MAX_IO4: U8.GPIO4
- new net MAX_IO5: U8.GPIO5
- new net MAX_IO6: U8.GPIO6
- new net MAX_IO7: U8.GPIO7
- new net MAX_IO8: U8.GPIO8
- new net MAX_IO9: U8.GPIO9
- new net N$1: U6.R, U8.RX1
- new net N$10: C13.1, U2.BOOT
- new net N$11: U4.D, U8.TX3
- new net N$12: U4.R, U8.RX3
- new net N$13: U7.DE, U7.~RE, U8.*RTS0
- new net N$14: U6.DE, U6.~RE, U8.*RTS1
- new net N$15: U5.DE, U5.~RE, U8.*RTS2
- new net N$16: U4.DE, U4.~RE, U8.*RTS3
- new net N$17: C1.1, R12.2, U8.*RST
- new net N$18: C2.1, U8.V18
- new net N$19: F4.1, T2.3, T4.3
- new net N$2: U5.D, U8.TX2
- new net N$20: D6.A, F4.2, R1.2
- new net N$3: U7.D, U8.TX0
- new net N$4: U5.R, U8.RX2
- new net N$5: U7.R, U8.RX0
- new net N$6: U6.D, U8.TX1
- new net N$7: R4.1, U2.RT/SYNC
- new net N$8: C9.2, R5.2, R6.1, U2.FB
- new net N$9: C13.2, D2.C, L1.2, U2.SW
- new net RPI_CS: A2.!CE0!/GPIO10, U8.*CS/A0
- new net RPI_IRQ: A2.GPIO0, R13.2, U8.*IRQ
- new net RPI_MISO: A2.GPIO13/MISO, U8.MISO/SDA
- new net RPI_MOSI: A2.GPIO12/MOSI, U8.MOSI/A1
- new net RPI_SCLK: A2.GPIO14/SCLK, U8.SCLK/SCL
Other:
- note added: "OSCILLATOR"
- note added: "RPI 3B+ HEADER"
- note added: "RS485"
- note added: "SPI TO UART"
- note added: "SUPPLY"
- note added: "TERMINALS"
